File: ignite-fidget-spinner.kicad_pcb (KiCad board)
At the start: 2 copper layers, 30 x 80 mm, 26 parts, among them Q3 2N3906, Q4 2N3904, Q5 2N3904, Q6 2N3904, SW1 SW Push 6mm

Commit message: Replace with simplified design
Parts:
- removed BT1, BT2: 1.5, Keystone_BAT_2997:BatteryHolder_Keystone_2997_LR44
- removed C1, C2, C3: 100n, Capacitor_THT:C_Disc_D5.1mm_W3.2mm_P5.00mm
- removed G***: LOGO, LOGO
- removed Q3: 2N3906, Package_TO_SOT_THT:TO-92_Inline
- removed Q4, Q5, Q6: 2N3904, Package_TO_SOT_THT:TO-92_Inline
- removed R1, R4, R5: 10k, Resistor_THT:R_Axial_DIN0207_L6.3mm_D2.5mm_P10.16mm_Horizontal
- removed R11, R2: 1k, Resistor_THT:R_Axial_DIN0207_L6.3mm_D2.5mm_P10.16mm_Horizontal
- removed R3: 1M, Resistor_THT:R_Axial_DIN0207_L6.3mm_D2.5mm_P10.16mm_Horizontal
- removed SW1: SW Push 6mm, Button_Switch_THT:SW_PUSH_6mm
- added D5: LED, LED_THT:LED_D3.0mm, F.Cu at (1.18, 24.1)
- R10, R6, R9: value 1k -> 470
- R7, R8: value 1M -> 470
- moved D4 107.1 mm to (1.18, 18.6), turned to 0 degrees
- moved D3 107.1 mm to (1.18, 13.2), turned to 0 degrees
- moved D2 107.1 mm to (1.18, 7.71), turned to 0 degrees
- moved D1 107.1 mm to (1.18, 2.23), turned to 0 degrees
- moved R6 98.4 mm to (6.96, 1.52), turned to 0 degrees
- moved R7 94.3 mm to (6.96, 5.58), turned to 0 degrees
- moved R8 93.7 mm to (6.96, 9.62), turned to 0 degrees
- moved R10 93.4 mm to (6.96, 17.7), turned to 0 degrees
- moved R9 90.0 mm to (6.96, 13.7), turned to 0 degrees
Connections:
- R10 pad 1: Net-(D3-K) -> Net-(D5-K)
- R10 pad 2: Net-(Q6-C) -> Net-(BT2--)
- R6 pad 2: Net-(Q5-C) -> Net-(BT2--)
- R7 pad 1: Net-(D1-A) -> Net-(D2-K)
- R7 pad 2: Net-(Q6-B) -> Net-(BT2--)
- R8 pad 1: Net-(D1-A) -> Net-(D3-K)
- R8 pad 2: Net-(Q5-B) -> Net-(BT2--)
- R9 pad 1: Net-(D2-K) -> Net-(D4-K)
- R9 pad 2: Net-(Q5-C) -> Net-(BT2--)
Routing:
- net Net-(D1-A): track 108.1 -> 0.00 mm, vias 1 -> 0
- net Net-(BT2--): track 84.6 -> 0.00 mm
- net Net-(BT1--): track 59.1 -> 0.00 mm
- net Net-(Q5-B): track 47.0 -> 0.00 mm
- net Net-(C1-Pad1): track 45.4 -> 0.00 mm
- net Net-(Q6-C): track 37.8 -> 0.00 mm, vias 1 -> 0
- net Net-(Q4-B): track 37.4 -> 0.00 mm
- net Net-(BT1-+): track 32.1 -> 0.00 mm
- net Net-(Q5-C): track 27.5 -> 0.00 mm
- net Net-(Q6-B): track 22.2 -> 0.00 mm
- net Net-(Q3-B): track 17.1 -> 0.00 mm
- net Net-(D2-K): track 10.4 -> 0.00 mm
- net Net-(D3-K): track 9.74 -> 0.00 mm
- net Net-(Q4-C): track 8.07 -> 0.00 mm
- net Net-(D4-K): track 5.54 -> 0.00 mm
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Other:
- board text removed: "Ignite Pre-O"
- board text removed: "LR44"

Commit message: Finish routing
Parts:
- added BT1: 1.5, Keystone_BAT_2997:BatteryHolder_Keystone_2997_LR44, F.Cu at (90.5, 52.5)
- added BT2: 1.5, Keystone_BAT_2997:BatteryHolder_Keystone_2997_LR44, F.Cu at (109.5, 97.5)
- added G***: LOGO, LOGO, F.Cu at (111.0, 75.0)
- added SW1: SW_SPDT, SW_SLW-864574-5A-RA-N-D:SW_SLW-864574-5A-RA-N-D, F.Cu at (112.0, 59.0)
- moved D1 145.4 mm to (98.7, 110.0)
- moved R1 133.3 mm to (91.0, 105.0)
- moved D3 130.6 mm to (98.7, 100.0)
- moved R3 119.8 mm to (91.0, 95.0)
- moved D5 117.7 mm to (98.7, 90.0)
- moved R4 108.3 mm to (109.0, 50.0), turned to 180 degrees
- moved R2 107.7 mm to (109.0, 40.0), turned to 180 degrees
- moved R5 107.6 mm to (91.0, 85.0)
- moved D2 106.8 mm to (101.3, 45.0), turned to 180 degrees
- moved D4 106.5 mm to (101.3, 55.0), turned to 180 degrees
- renumbered R6 to R1, R7 to R2, R8 to R3, R9 to R4, R10 to R5
Routing:
- net Net-(BT2--): track 0.00 -> 78.2 mm
- net Net-(D1-A): track 0.00 -> 72.6 mm
- net Net-(BT1--): track 0.00 -> 64.0 mm
- net Net-(BT1-+): track 0.00 -> 41.0 mm
- net Net-(D5-K): track 0.00 -> 9.80 mm
- net Net-(D3-K): track 0.00 -> 9.80 mm
- net Net-(D2-K): track 0.00 -> 9.80 mm
- net Net-(D1-K): track 0.00 -> 9.80 mm
- net Net-(D4-K): track 0.00 -> 9.80 mm
Other:
- board text added: "Clarkson Ignite Pre-O"
- board text added: "Designed in 2025 by Sigmond Kukla & Elizabeth Kraynak"

Commit message: Finish aesthetics
Parts:
- added kibuzzard-6892C1DC: G***, kibuzzard-6892C1DC, F.Cu at (87.8, 81.5)
- added kibuzzard-6892C246: G***, kibuzzard-6892C246, F.Cu at (108.5, 60.0)
- added kibuzzard-6892C379: G***, kibuzzard-6892C379, B.Cu at (113.0, 97.5)
- added kibuzzard-6892C379: G***, kibuzzard-6892C379, B.Cu at (87.0, 52.5)
- R1, R2, R3, R4, R5: value 470 -> 220
- moved SW1 1.12 mm to (112.5, 60.0)
Routing:
- net Net-(BT1-+): track 41.0 -> 43.7 mm
- net Net-(D1-A): track 72.6 -> 73.9 mm
Other:
- outline, holes or cut-outs redrawn
- board text added: "-"
- board text added: "- +"
- board text added: "1.5V LR44"
- board text added: "JLCJLCJLCJLC"
- board text removed: "Clarkson Ignite Pre-O"
